Commit message: Added proper wheel joints to the URDF
Changelog: None
Signed-off-by: Ole Petter <ole.orhagen@northern.tech>

File: urdf/r2d2.urdf (robot description, URDF)
Before this commit: robot r2d2, 7 links, 6 joints
Joints:
- joint joint_left_back_wheel: axis (none) -> 1 0 0; origin (none) -> xyz=-0.35 -0.4 0
- joint joint_left_front_wheel: axis (none) -> 1 0 0; origin (none) -> xyz=-0.35 0.4 0
- joint joint_right_back_wheel: axis (none) -> 1 0 0; origin (none) -> xyz=0.35 -0.4 0
- joint joint_right_front_wheel: axis (none) -> 1 0 0; origin (none) -> xyz=0.35 0.4 0.0

Commit message: Add collision detection to the model
Changelog: None
Signed-off-by: Ole Petter <ole.orhagen@northern.tech>

File: urdf/r2d2.urdf (robot description, URDF)
Before this commit: robot r2d2, 7 links, 6 joints
Links:
- link back_suspension: geometry collision cylinder length=0.7 radius=0.1; visual cylinder length=0.7 radius=0.1
- link base_link: geometry collision box size=0.5 1.0 0.3; visual box size=0.5 1.0 0.3
- link front_suspension: geometry collision cylinder length=0.7 radius=0.1; visual cylinder length=0.7 radius=0.1
- link left_back_wheel: geometry collision cylinder length=0.1 radius=0.2; visual cylinder length=0.1 radius=0.2
- link left_front_wheel: geometry collision cylinder length=0.1 radius=0.2; visual cylinder length=0.1 radius=0.2
- link right_back_wheel: geometry collision cylinder length=0.1 radius=0.2; visual cylinder length=0.1 radius=0.2
- link right_front_wheel: geometry collision cylinder length=0.1 radius=0.2; visual cylinder length=0.1 radius=0.2

Commit message: Add inertia to the main links in the URDF
Changelog: None
Signed-off-by: Ole Petter <ole.orhagen@northern.tech>

File: urdf/r2d2.urdf (robot description, URDF)
Before this commit: robot r2d2, 7 links, 6 joints
Links:
- link base_link: mass None -> 2.0
- link left_back_wheel: mass None -> 0.2
- link left_front_wheel: mass None -> 0.2
- link right_back_wheel: mass None -> 0.2
- link right_front_wheel: mass None -> 0.2

Commit message: Add chassis link
Changelog: None
Signed-off-by: Ole Petter <ole.orhagen@northern.tech>

File: urdf/r2d2.urdf (robot description, URDF)
Before this commit: robot r2d2, 7 links, 6 joints
Links:
- added link chassis, mass 2.0; collision box size=0.5 1.0 0.3; visual box size=0.5 1.0 0.3
- link base_link: mass 2.0 -> None; geometry 
Joints:
- added joint chassis_to_base_link: type fixed, parent base_link, child chassis

Commit message: Added ackermann steering front-wheels to the URDF
Changelog: None
Signed-off-by: Ole Petter <ole.orhagen@northern.tech>

File: urdf/r2d2.urdf (robot description, URDF)
Before this commit: robot r2d2, 8 links, 7 joints
Links:
- added link front_left_steer_bar; visual cylinder length=0.1 radius=0.01
- added link front_right_steer_bar; visual cylinder length=0.1 radius=0.01
Joints:
- added joint joint_front_left_steer_bar: type revolute, parent chassis, child front_left_steer_bar, origin xyz=-0.35 0.40 0.0, axis 0 0 1, limit lower=-0.1 upper=0.1 effort=100 velocity=10
- added joint joint_front_right_steer_bar: type revolute, parent chassis, child front_right_steer_bar, origin xyz=0.35 0.40 0.0, axis 0 0 1, limit lower=-0.1 upper=0.1 effort=100 velocity=10
- joint joint_left_front_wheel: origin xyz=-0.35 0.4 0 -> xyz=0.0 0.0 0.0; parent base_link -> front_left_steer_bar
- joint joint_right_front_wheel: origin xyz=0.35 0.4 0.0 -> xyz=0.0 0.0 0.0; parent base_link -> front_right_steer_bar

Commit message: Extend front-wheel turning angle to 0.3
Changelog: None
Signed-off-by: Ole Petter <ole.orhagen@northern.tech>

File: urdf/r2d2.urdf (robot description, URDF)
Before this commit: robot r2d2, 10 links, 9 joints
Joints:
- joint joint_front_left_steer_bar: limit lower=-0.1 upper=0.1 effort=100 velocity=10 -> lower=-0.3 upper=0.3 effort=100 velocity=10
- joint joint_front_right_steer_bar: limit lower=-0.1 upper=0.1 effort=100 velocity=10 -> lower=-0.3 upper=0.3 effort=100 velocity=10

Commit message: Change chassis as the new base for the dependent links
Changelog: None
Signed-off-by: Ole Petter <ole.orhagen@northern.tech>

File: urdf/r2d2.urdf (robot description, URDF)
Before this commit: robot r2d2, 10 links, 9 joints
Joints:
- joint back_suspension_to_base_link: parent base_link -> chassis
- joint front_suspension_to_base_link: parent base_link -> chassis

Commit message: Add inertial tags to the steer joints
Changelog: None
Signed-off-by: Ole Petter <ole.orhagen@northern.tech>

File: urdf/r2d2.urdf (robot description, URDF)
Before this commit: robot r2d2, 10 links, 9 joints
Links:
- link front_left_steer_bar: mass None -> 0.01
- link front_right_steer_bar: mass None -> 0.01

Commit message: Link to the chassis, instead of the base_link
Changelog: None
Signed-off-by: Ole Petter <ole.orhagen@northern.tech>

File: urdf/r2d2.urdf (robot description, URDF)
Before this commit: robot r2d2, 10 links, 9 joints
Joints:
- joint joint_left_back_wheel: parent base_link -> chassis
- joint joint_right_back_wheel: parent base_link -> chassis

Commit message: Don't allow any effort on the front wheels
Changelog: None
Signed-off-by: Ole Petter <ole.orhagen@northern.tech>

File: urdf/r2d2.urdf (robot description, URDF)
Before this commit: robot r2d2, 10 links, 9 joints
Joints:
- joint joint_left_front_wheel: limit (none) -> lower=-0.3 upper=0.3 effort=0.0 velocity=10
- joint joint_right_front_wheel: limit (none) -> lower=-0.3 upper=0.3 effort=0.0 velocity=10

Commit message: Add a Lidar to the simulated vehicle
Changelog: None
Signed-off-by: Ole Petter <ole.orhagen@northern.tech>

File: urdf/r2d2.urdf (robot description, URDF)
Before this commit: robot r2d2, 10 links, 9 joints
Links:
- added link lidar_cylinder, mass 0.2; collision cylinder length=0.1 radius=0.1; visual cylinder length=0.1 radius=0.1
Joints:
- added joint joint_lidar_cylinder: type fixed, parent chassis, child lidar_cylinder, origin xyz=0 0 0.2

Commit message: Add a camera to the front of the vehicle
Changelog: None
Signed-off-by: Ole Petter <ole.orhagen@northern.tech>

File: urdf/r2d2.urdf (robot description, URDF)
Before this commit: robot r2d2, 11 links, 10 joints
Links:
- added link camera_box, mass 0.1; collision box size=0.05 0.05 0.05; visual box size=0.05 0.05 0.05
Joints:
- added joint joint_camera_box: type fixed, parent chassis, child camera_box, origin xyz=0 0.5 0 rpy=0 0 ${pi/2}

Commit message: Move the URDF to a single front-wheel steer
Changelog: None
Signed-off-by: Ole Petter <ole.orhagen@northern.tech>

File: urdf/r2d2.urdf (robot description, URDF)
Before this commit: robot r2d2, 12 links, 11 joints
Links:
- removed link front_left_steer_bar
- removed link front_right_steer_bar
- removed link front_suspension
- removed link left_front_wheel
- removed link right_front_wheel
- added link front_steer_bar, mass 0.01; visual cylinder length=0.1 radius=0.01
- added link front_wheel, mass 0.2; collision cylinder length=0.1 radius=0.2; visual cylinder length=0.1 radius=0.2
Joints:
- removed joint front_suspension_to_base_link
- removed joint joint_front_left_steer_bar
- removed joint joint_front_right_steer_bar
- removed joint joint_left_front_wheel
- removed joint joint_right_front_wheel
- added joint joint_front_steer_bar: type revolute, parent chassis, child front_steer_bar, origin xyz=0.0 0.40 0.0, axis 0 0 1, limit lower=-0.3 upper=0.3 effort=100 velocity=10
- added joint joint_front_wheel: type continuous, parent front_steer_bar, child front_wheel, origin xyz=0.0 0.0 0.0, axis 1 0 0, limit lower=-0.3 upper=0.3 effort=0.0 velocity=10

Commit message: Change the position and height of the lidar sensor
Changelog: None
Signed-off-by: Ole Petter <ole.orhagen@northern.tech>

File: urdf/r2d2.urdf (robot description, URDF)
Before this commit: robot r2d2, 9 links, 8 joints
Links:
- link lidar_cylinder: geometry collision cylinder length=0.2 radius=0.1; visual cylinder length=0.2 radius=0.1
Joints:
- joint joint_lidar_cylinder: origin xyz=0 0 0.2 -> xyz=0 0 0.3

Commit message: Started using xacro in the URDF
Changelog: None
Signed-off-by: Ole Petter <ole.orhagen@northern.tech>

File: urdf/r2d2.urdf (robot description, URDF)
Before this commit: robot r2d2, 9 links, 8 joints
Links:
- removed link chassis
Joints:
- removed joint chassis_to_base_link

Commit message: Redrew the robot to face in the x-direction
Changelog: None
Signed-off-by: Ole Petter <ole.orhagen@northern.tech>

File: urdf/r2d2.urdf (robot description, URDF)
Before this commit: robot r2d2, 8 links, 7 joints
Links:
- removed link back_suspension
- removed link front_steer_bar
- removed link front_wheel
- removed link left_back_wheel
- removed link right_back_wheel
Joints:
- removed joint back_suspension_to_base_link
- joint joint_camera_box: origin xyz=0 0.5 0 rpy=0 0 ${pi/2} -> xyz=0.5 0.0 0 rpy=0 0 0
- joint joint_front_steer_bar: origin xyz=0.0 0.40 0.0 -> xyz=${chassis_xsize/2 - wheel_radius} 0 ${wheel_radius/4}
- joint joint_front_wheel: axis 1 0 0 -> 0 1 0; origin xyz=0.0 0.0 0.0 -> xyz=${chassis_xsize/2 - wheel_radius} 0 ${-chassis_zsize/4}
- joint joint_left_back_wheel: axis 1 0 0 -> 0 1 0; limit (none) -> lower=-0.3 upper=0.3 effort=100 velocity=10; origin xyz=-0.35 -0.4 0 -> xyz=${-chassis_xsize/2 + wheel_radius/2} ${chassis_ysize/2 + 0.1} ${-chassis_zsize/4}
- joint joint_right_back_wheel: axis 1 0 0 -> 0 1 0; limit (none) -> lower=-0.3 upper=0.3 effort=100 velocity=10; origin xyz=0.35 -0.4 0 -> xyz=${-chassis_xsize/2 + wheel_radius/2} ${-chassis_ysize/2 - 0.1} ${-chassis_zsize/4}

Commit message: Added 4 wheels back into the URDF model
Changelog: None
Signed-off-by: Ole Petter <ole.orhagen@northern.tech>

File: urdf/r2d2.urdf (robot description, URDF)
Before this commit: robot r2d2, 3 links, 6 joints
Joints:
- added joint joint_left_front_wheel: type continuous, parent chassis, child left_front_wheel, origin xyz=${chassis_xsize/2 - wheel_radius/2} ${chassis_ysize/2 + 0.1} ${axel_zpos}, axis 0 1 0, limit lower=-0.3 upper=0.3 effort=100 velocity=10
- added joint joint_right_front_wheel: type continuous, parent chassis, child right_front_wheel, origin xyz=${chassis_xsize/2 - wheel_radius/2} ${-chassis_ysize/2 - 0.1} ${axel_zpos}, axis 0 1 0, limit lower=-0.3 upper=0.3 effort=100 velocity=10
- joint joint_front_steer_bar: origin xyz=${chassis_xsize/2 - wheel_radius} 0 ${wheel_radius/4} -> xyz=${front_axel_xpos} 0 ${axel_zpos}
- joint joint_front_wheel: origin xyz=${chassis_xsize/2 - wheel_radius} 0 ${-chassis_zsize/4} -> (none)
- joint joint_left_back_wheel: origin xyz=${-chassis_xsize/2 + wheel_radius/2} ${chassis_ysize/2 + 0.1} ${-chassis_zsize/4} -> xyz=${-chassis_xsize/2 + wheel_radius/2} ${chassis_ysize/2 + 0.1} ${axel_zpos}
- joint joint_right_back_wheel: mimic (none) -> joint=joint_left_back_wheel; origin xyz=${-chassis_xsize/2 + wheel_radius/2} ${-chassis_ysize/2 - 0.1} ${-chassis_zsize/4} -> xyz=${-chassis_xsize/2 + wheel_radius/2} ${-chassis_ysize/2 - 0.1} ${axel_zpos}

Commit message: Parameterized the car construction in the URDF
Changelog: None
Signed-off-by: Ole Petter <ole.orhagen@northern.tech>

File: urdf/r2d2.urdf (robot description, URDF)
Before this commit: robot r2d2, 3 links, 8 joints
Joints:
- joint joint_left_back_wheel: origin xyz=${-chassis_xsize/2 + wheel_radius/2} ${chassis_ysize/2 + 0.1} ${axel_zpos} -> xyz=${back_axel_xpos} ${-axel_width/2} ${axel_zpos}
- joint joint_left_front_wheel: origin xyz=${chassis_xsize/2 - wheel_radius/2} ${chassis_ysize/2 + 0.1} ${axel_zpos} -> xyz=${front_axel_xpos} ${-axel_width/2} ${axel_zpos}
- joint joint_right_back_wheel: origin xyz=${-chassis_xsize/2 + wheel_radius/2} ${-chassis_ysize/2 - 0.1} ${axel_zpos} -> xyz=${back_axel_xpos} ${axel_width/2} ${axel_zpos}
- joint joint_right_front_wheel: origin xyz=${chassis_xsize/2 - wheel_radius/2} ${-chassis_ysize/2 - 0.1} ${axel_zpos} -> xyz=${front_axel_xpos} ${axel_width/2} ${axel_zpos}

Commit message: Ready Rviz URDF of the four wheel car
Changelog: None
Signed-off-by: Ole Petter <ole.orhagen@northern.tech>

File: urdf/r2d2.urdf (robot description, URDF)
Before this commit: robot r2d2, 3 links, 8 joints
Joints:
- added joint joint_left_front_steer_bar: type revolute, parent chassis, child left_front_steer_bar, origin xyz=${front_axel_xpos} ${axel_width/2} ${axel_zpos}, axis 0 0 1, limit lower=-0.3 upper=0.3 effort=100 velocity=10
- added joint joint_right_front_steer_bar: type revolute, parent chassis, child right_front_steer_bar, origin xyz=${front_axel_xpos} ${-axel_width/2} ${axel_zpos}, axis 0 0 1, limit lower=-0.3 upper=0.3 effort=100 velocity=10
- joint joint_left_back_wheel: origin xyz=${back_axel_xpos} ${-axel_width/2} ${axel_zpos} -> xyz=${back_axel_xpos} ${axel_width/2} ${axel_zpos}
- joint joint_left_front_wheel: limit lower=-0.3 upper=0.3 effort=100 velocity=10 -> lower=-0.3 upper=0.3 effort=0 velocity=10; origin xyz=${front_axel_xpos} ${-axel_width/2} ${axel_zpos} -> (none); parent chassis -> left_front_steer_bar
- joint joint_right_back_wheel: origin xyz=${back_axel_xpos} ${axel_width/2} ${axel_zpos} -> xyz=${back_axel_xpos} ${-axel_width/2} ${axel_zpos}
- joint joint_right_front_wheel: limit lower=-0.3 upper=0.3 effort=100 velocity=10 -> lower=-0.3 upper=0.3 effort=0 velocity=10; origin xyz=${front_axel_xpos} ${axel_width/2} ${axel_zpos} -> (none); parent chassis -> right_front_steer_bar

Commit message: Added a controller from the steer_bot (not working atm)
Changelog: None
Signed-off-by: Ole Petter <ole.orhagen@northern.tech>

File: urdf/r2d2.urdf (robot description, URDF)
Before this commit: robot r2d2, 3 links, 10 joints
Joints:
- added joint joint_back_wheel: type continuous, parent chassis, child back_wheel, origin xyz=${back_axel_xpos} 0 ${axel_zpos}, axis 0 1 0, limit lower=-0.3 upper=0.3 effort=100 velocity=10

Commit message: Add: xacro:properties for the wheel efforts and speeds
Changelog: None
Signed-off-by: Ole Petter <ole.orhagen@northern.tech>

File: urdf/r2d2.urdf (robot description, URDF)
Before this commit: robot r2d2, 3 links, 11 joints
Joints:
- joint joint_back_wheel: limit lower=-0.3 upper=0.3 effort=100 velocity=10 -> effort=${wheel_speed_effort} velocity=${wheel_speed_velocity}
- joint joint_front_steer_bar: limit lower=-0.3 upper=0.3 effort=100 velocity=10 -> lower=-${wheel_swing_limit} upper=${wheel_swing_limit} effort=${wheel_swing_effort} velocity=${wheel_swing_velocity}
- joint joint_front_wheel: limit lower=-0.3 upper=0.3 effort=0.0 velocity=10 -> effort=${wheel_speed_effort} velocity=${wheel_speed_velocity}
- joint joint_left_back_wheel: limit lower=-0.3 upper=0.3 effort=100 velocity=10 -> effort=${wheel_speed_effort} velocity=${wheel_speed_velocity}
- joint joint_left_front_steer_bar: limit lower=-0.3 upper=0.3 effort=100 velocity=10 -> lower=${-wheel_swing_limit} upper=${wheel_swing_limit} effort=${wheel_swing_effort} velocity=${wheel_swing_velocity}
- joint joint_left_front_wheel: limit lower=-0.3 upper=0.3 effort=0 velocity=10 -> effort=0 velocity=10
- joint joint_right_back_wheel: limit lower=-0.3 upper=0.3 effort=100 velocity=10 -> effort=${wheel_speed_effort} velocity=${wheel_speed_velocity}
- joint joint_right_front_steer_bar: limit lower=-0.3 upper=0.3 effort=100 velocity=10 -> lower=${-wheel_swing_limit} upper=${wheel_swing_limit} effort=${wheel_swing_limit} velocity=${wheel_swing_velocity}
- joint joint_right_front_wheel: limit lower=-0.3 upper=0.3 effort=0 velocity=10 -> effort=0 velocity=10

Commit message: Give the steer bar some mass
Changelog: None
Signed-off-by: Ole Petter <ole.orhagen@northern.tech>

File: urdf/r2d2.urdf (robot description, URDF)
Before this commit: robot r2d2, 3 links, 11 joints
Joints:
- joint joint_front_wheel: limit effort=${wheel_speed_effort} velocity=${wheel_speed_velocity} -> effort=0 velocity=10
- joint joint_left_front_steer_bar: limit lower=${-wheel_swing_limit} upper=${wheel_swing_limit} effort=${wheel_swing_effort} velocity=${wheel_swing_velocity} -> lower=${-wheel_swing_limit} upper=${wheel_swing_limit} effort=${wheel_swing_limit} velocity=${wheel_swing_velocity}
